Commit message: Update gripper xacro and add control guide

File: indy_openvla/urdf/indy.ros2_control.xacro (robot description, xacro)
@@ -55,6 +55,4 @@
             </joint>
             <joint name="${prefix}right_finger_joint">
-                <param name="mimic">${prefix}left_finger_joint</param>
-                <param name="multiplier">1.0</param>
                 <command_interface name="position">
                     <param name="min">0.0</param>

File: indy_openvla/urdf/indy_gripper.xacro (robot description, xacro)
@@ -19,5 +19,5 @@
                 <origin xyz="0 0 ${gripper_body_length/2}" rpy="0 0 0"/>
                 <geometry>
-                    <box size="${gripper_body_length} ${finger_spread + finger_width*2} ${gripper_body_length}"/>
+                    <box size="${gripper_body_length} ${finger_spread + finger_width*2 + 0.06} ${gripper_body_length}"/>
                 </geometry>
                 <material name="gripper_metal_grey"/>
@@ -26,5 +26,5 @@
                 <origin xyz="0 0 ${gripper_body_length/2}" rpy="0 0 0"/>
                 <geometry>
-                    <box size="${gripper_body_length} ${finger_spread + finger_width*2} ${gripper_body_length}"/>
+                    <box size="${gripper_body_length} ${finger_spread + finger_width*2 + 0.06} ${gripper_body_length}"/>
                 </geometry>
             </collision>
