Commit message: Feat: Add MoveIt integration and dual controller setup

File: indy_openvla/urdf/indy_gripper.xacro (robot description, xacro)
@@ -88,7 +88,4 @@
             <safety_controller soft_lower_limit="0.0" soft_upper_limit="${max_opening/2}" k_position="100" k_velocity="1"/>
         </joint>
-        <gazebo reference="${prefix}right_finger_joint">
-            <mimic joint="${prefix}left_finger_joint" multiplier="1" offset="0"/>
-        </gazebo>
     </xacro:macro>
 </robot>

Commit message: feat: Add YOLO vision-based autonomous grasping

File: indy_openvla/urdf/indy_gripper.xacro (robot description, xacro)
@@ -9,15 +9,15 @@
     <xacro:macro name="indy_two_finger_gripper" params="prefix parent_link tcp_offset_xyz">
         <xacro:property name="gripper_mass" value="0.5" />
-        <xacro:property name="finger_length" value="0.10" />
+        <xacro:property name="finger_length" value="0.12" />
         <xacro:property name="finger_width" value="0.015" />
-        <xacro:property name="finger_depth" value="0.015" />
+        <xacro:property name="finger_depth" value="0.04" />
         <xacro:property name="gripper_body_length" value="0.06" />
-        <xacro:property name="max_opening" value="0.08" />
-        <xacro:property name="finger_spread" value="0.04" />
+        <xacro:property name="max_opening" value="0.12" />
+        <xacro:property name="finger_spread" value="0.06" />
         <link name="${prefix}gripper_base_link">
             <visual>
                 <origin xyz="0 0 ${gripper_body_length/2}" rpy="0 0 0"/>
                 <geometry>
-                    <box size="${gripper_body_length} ${finger_spread + finger_width*2 + 0.06} ${gripper_body_length}"/>
+                    <box size="${gripper_body_length} ${finger_spread + finger_width*2 + 0.14} ${gripper_body_length}"/>
                 </geometry>
                 <material name="gripper_metal_grey"/>
@@ -26,5 +26,5 @@
                 <origin xyz="0 0 ${gripper_body_length/2}" rpy="0 0 0"/>
                 <geometry>
-                    <box size="${gripper_body_length} ${finger_spread + finger_width*2 + 0.06} ${gripper_body_length}"/>
+                    <box size="${gripper_body_length} ${finger_spread + finger_width*2 + 0.14} ${gripper_body_length}"/>
                 </geometry>
             </collision>
@@ -42,10 +42,10 @@
         <link name="${prefix}left_finger_link">
              <visual>
-                <origin xyz="0 ${finger_width/2} 0" rpy="0 0 0"/>
+                <origin xyz="0 ${finger_width/2} ${finger_length/2}" rpy="0 0 0"/>
                 <geometry><box size="${finger_depth} ${finger_width} ${finger_length}"/></geometry>
                 <material name="gripper_metal"/>
             </visual>
             <collision>
-                <origin xyz="0 ${finger_width/2} 0" rpy="0 0 0"/>
+                <origin xyz="0 ${finger_width/2} ${finger_length/2}" rpy="0 0 0"/>
                 <geometry><box size="${finger_depth} ${finger_width} ${finger_length}"/></geometry>
             </collision>
@@ -66,10 +66,10 @@
         <link name="${prefix}right_finger_link">
             <visual>
-                <origin xyz="0 ${-finger_width/2} 0" rpy="0 0 0"/>
+                <origin xyz="0 ${-finger_width/2} ${finger_length/2}" rpy="0 0 0"/>
                 <geometry><box size="${finger_depth} ${finger_width} ${finger_length}"/></geometry>
                 <material name="gripper_metal"/>
             </visual>
             <collision>
-                <origin xyz="0 ${-finger_width/2} 0" rpy="0 0 0"/>
+                <origin xyz="0 ${-finger_width/2} ${finger_length/2}" rpy="0 0 0"/>
                 <geometry><box size="${finger_depth} ${finger_width} ${finger_length}"/></geometry>
             </collision>

File: indy_openvla/urdf/indy_macro.xacro (robot description, xacro)
@@ -230,5 +230,5 @@
                 <parent link="${prefix}link6"/>
                 <child link="${prefix}zed2i_camera_link"/>
-                <origin xyz="0.08 0 0" rpy="0 0 -1.5708"/>
+                <origin xyz="-0.08 0 0" rpy="0 0 1.5708"/>
             </joint>
             <link name="${prefix}zed2i_camera_frame"/>
