Commit message: Feat: Update README

File: indy_moveit/srdf/indy_macro.srdf.xacro (robot description, xacro)
@@ -12,6 +12,18 @@
         <!--SUBGROUPS - Groups can also be formed by referencing to already defined group names-->
         <group name="${prefix}${name}_manipulator">
-            <chain base_link="${prefix}link0" tip_link="${prefix}tcp" />
+            <chain base_link="${prefix}link0" tip_link="${prefix}link6" />
         </group>
+        <group name="${prefix}gripper">
+            <joint name="${prefix}left_finger_joint" />
+            <joint name="${prefix}right_finger_joint" />
+        </group>
+        <group_state name="${prefix}gripper_open" group="${prefix}gripper">
+            <joint name="${prefix}left_finger_joint" value="0.06" />
+            <joint name="${prefix}right_finger_joint" value="0.06" />
+        </group_state>
+        <group_state name="${prefix}gripper_closed" group="${prefix}gripper">
+            <joint name="${prefix}left_finger_joint" value="0.0" />
+            <joint name="${prefix}right_finger_joint" value="0.0" />
+        </group_state>
         <xacro:if value="${indy_type == 'indyrp2' or indy_type == 'indyrp2_v2'}">
             <!--GROUP STATES - Purpose - Define a named state for a particular group, in terms of joint values. This is useful to define states like 'folded arms'-->
@@ -23,4 +35,13 @@
                 <joint name="${prefix}joint4" value="0" />
                 <joint name="${prefix}joint5" value="-1.570796327" />
+                <joint name="${prefix}joint6" value="0" />
+            </group_state>
+            <group_state name="${prefix}Ready" group="${prefix}${name}_manipulator">
+                <joint name="${prefix}joint0" value="0.4189" />
+                <joint name="${prefix}joint1" value="-0.1571" />
+                <joint name="${prefix}joint2" value="-1.3963" />
+                <joint name="${prefix}joint3" value="0" />
+                <joint name="${prefix}joint4" value="-1.5882" />
+                <joint name="${prefix}joint5" value="0.4189" />
                 <joint name="${prefix}joint6" value="0" />
             </group_state>
@@ -56,4 +77,12 @@
                 <joint name="${prefix}joint5" value="0" />
             </group_state>
+            <group_state name="${prefix}Ready" group="${prefix}${name}_manipulator">
+                <joint name="${prefix}joint0" value="0.4189" />
+                <joint name="${prefix}joint1" value="-0.1571" />
+                <joint name="${prefix}joint2" value="-1.3963" />
+                <joint name="${prefix}joint3" value="0" />
+                <joint name="${prefix}joint4" value="-1.5882" />
+                <joint name="${prefix}joint5" value="0.4189" />
+            </group_state>
             <group_state name="${prefix}ZeroPos" group="${prefix}${name}_manipulator">
                 <joint name="${prefix}joint0" value="0" />
@@ -80,4 +109,9 @@
             <disable_collisions link1="link3" link2="link6" reason="Never" />
             <disable_collisions link1="link4" link2="link6" reason="Never" />
+            <!-- Gripper collision disabling -->
+            <disable_collisions link1="${prefix}link6" link2="${prefix}gripper_base_link" reason="Adjacent" />
+            <disable_collisions link1="${prefix}gripper_base_link" link2="${prefix}left_finger_link" reason="Adjacent" />
+            <disable_collisions link1="${prefix}gripper_base_link" link2="${prefix}right_finger_link" reason="Adjacent" />
+            <disable_collisions link1="${prefix}left_finger_link" link2="${prefix}right_finger_link" reason="Never" />
         </xacro:unless>
     </xacro:macro>
